File: ControlModule.sch (EAGLE design)
At the start: 2 parts, among them U1 ATMEGA328P

Commit message: drawing Control Module
Parts:
- added IC1, IC2: (no value), v-reg:LM138-TL
- added PAD1, PAD10, PAD11, PAD2, PAD3, PAD4, PAD5, PAD6, PAD7, PAD8, PAD9: (no value), wirepad:2,54/1,1
- added R1: (no value), rcl:R-EU_R0805
Connections:
- new net 0: IC1.ADJ, IC2.ADJ, PAD2.P, PAD4.P, PAD7.P, PAD8.P, R1.1, U$1.24-GND, U1.GND@2
- new net BATT: U$1.23-VDD, U1.VCC
- new net IN1: PAD9.P, U1.PC0(ADC0)
- new net IN2: PAD10.P, U1.PC1(ADC1)
- new net IN3: PAD11.P, U1.PC2(ADC2)
- new net N$1: U$1.6-RX, U1.PD1(TXD)
- new net N$2: U$1.5-TX, U1.PD0(RXD)
- new net N$3: U$1.14-CTS-PIO5, U1.PD2(INT0)
- new net N$4: U$1.18-RTS-PIO6, U1.PD3(INT1)
- new net N$5: IC1.IN, PAD1.P
- new net N$6: IC2.IN, PAD3.P
- new net N$7: IC1.OUT, PAD5.P
- new net N$9: IC2.OUT, PAD6.P
- new net PIO1: U$1.10-PIO1-SCK, U1.PB1(OC1A)
- new net PIO3: U$1.12-WS-PIO3-MOSI, U1.PB0(ICP)
- new net WAKEHW: U$1.15-WAKEHW, U1.PC5(ADC5/SCL)
- new net WAKESW: R1.2, U$1.7-WAKESW, U1.PC4(ADC4/SDA)
Other:
- moved on the sheet: U1

Commit message: Control module first version and Processing module final design
Parts:
- added 3V, GND: (no value), wirepad:2,54/1,1
- added C1, C2: 22pF, rcl:C-EUC0603
- added C3: (no value), rcl:C-EUC0603
- added C4, C5: 100nF, rcl:C-EUC0603
- added LED2: (no value), led:LEDCHIPLED_0603
- added PAD12: VREF, wirepad:2,54/1,1
- added Q1: 16MHz, crystal:CRYSTALHC49S
- added R2, R4: 10k, rcl:R-EU_R0805
- added R3: 220, rcl:R-EU_R0805
- added S1, S2: (no value), switch-omron:10-XX
- PAD1, PAD3: value (none) -> 9V
- PAD2, PAD4: value (none) -> GND
- PAD5: value (none) -> +6V
- PAD6, PAD7: value (none) -> AGND
- PAD8: value (none) -> -6V
- R1: value (none) -> 10k
Connections:
- net N$5 renamed 9V
- removed net BATT: U$1.23-VDD, U1.VCC
- removed net N$4: U$1.18-RTS-PIO6, U1.PD3(INT1)
- new net 3V: C3.2, C4.2, C5.2, R2.2, S2.S, U$1.23-VDD, U1.AVCC, U1.VCC
- new net CTS: U$1.14-CTS-PIO5, U1.PB1(OC1A)
- new net MLDP: U$1.8-CMD-MLDP, U1.PD4(XCK/T0)
- new net N$10: R2.1, S1.S, U1.PC6(/RESET)
- new net N$11: LED2.A, R3.1
- new net N$12: R4.2, S2.S1
- new net N$5: C1.2, Q1.2, U1.PB6(XTAL1/TOSC1)
- new net N$8: C2.2, Q1.1, U1.PB7(XTAL2/TOSC2)
- new net PIO2: U$1.11-MLDPEV-PIO2-CS, U1.PB4(MISO)
- new net RTS: U$1.18-RTS-PIO6, U1.PB2(SS/OC1B)
- net 0: now also C1.1, C2.1, C3.1, C4.1, C5.1, LED2.C, R4.1, S1.P, U$1.1-GND, U1.GND@1
- net N$1: now also U1.PD6(AIN0); no longer U1.PD1(TXD)
- net N$2: now also U1.PD5(T1); no longer U1.PD0(RXD)
- net N$3: now also S2.P, U1.PC3(ADC3); no longer U$1.14-CTS-PIO5, U1.PD2(INT0)
- net PIO1: now also R3.2, U1.PB5(SCK); no longer U1.PB1(OC1A)
- net WAKEHW: now also U1.PD3(INT1); no longer U1.PC5(ADC5/SCL)
- net WAKESW: now also U1.PD2(INT0); no longer U1.PC4(ADC4/SDA)
Other:
- moved on the sheet: IC1, IC2, PAD1, PAD10, PAD11, PAD2, PAD3, PAD4, PAD5, PAD6, PAD7, PAD8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
