File: ProcessingModule.brd (EAGLE design)
At the start: 35.5 x 43.1 mm, 32 parts, among them IC1 INA128U, IC2 LM358MX, IC3 MCP606-I_SN

Commit message: Control module first version and Processing module final design
Parts:
- added R6_2: 50k, rcl:R0805
Connections:
- net N$11: now also R6_2.2
- net N$4: now also R6_2.1
Routing:
- net N$11: track 24.4 -> 27.8 mm
- net N$4: track 27.1 -> 30.4 mm
- net AGND: track 139.2 -> 141.5 mm
Changed lines of the file:
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@@
 <attribute name="VALUE" x="11.049" y="5.588" size="1.27" layer="27" rot="R180"/>
+</element>
+<element name="R6_2" library="rcl" library_urn="urn:adsk.eagle:library:334" package="R0805" package3d_urn="urn:adsk.eagle:package:23553/2" value="50k" x="26.416" y="36.068">
+<attribute name="SPICEPREFIX" value="R" x="26.416" y="36.068" size="1.778" layer="27" display="off"/>
 </element>
 </elements>
@@
 <contactref element="PAD5" pad="1"/>
 <wire x1="3.8354" y1="32.385" x2="3.81" y2="32.678" width="0.4064" layer="1"/>
-<via x="3.81" y="29.464" extent="1-16" drill="0.8"/>
+<via x="3.81" y="29.464" extent="1-16" drill="1"/>
 <wire x1="3.81" y1="29.464" x2="3.81" y2="32.678" width="0.4064" layer="1"/>
 <wire x1="9.652" y1="24.042" x2="9.398" y2="24.296" width="0.4064" layer="1"/>
@@
 <wire x1="9.398" y1="24.296" x2="9.652" y2="24.55" width="0.4064" layer="1"/>
 <wire x1="9.398" y1="24.296" x2="11.51395" y2="24.296" width="0.4064" layer="1"/>
-<via x="23.114" y="25.654" extent="1-16" drill="0.8"/>
+<via x="23.114" y="25.654" extent="1-16" drill="1"/>
 <wire x1="25.466" y1="25.654" x2="23.114" y2="25.654" width="0.4064" layer="1"/>
 <wire x1="20.762" y1="25.654" x2="23.114" y2="25.654" width="0.4064" layer="1"/>
-<via x="30.226" y="21.082" extent="1-16" drill="0.8"/>
+<via x="30.226" y="21.082" extent="1-16" drill="1"/>
 <wire x1="5.334" y1="18.796" x2="3.81" y2="20.32" width="0.4064" layer="1"/>
 <wire x1="3.81" y1="29.464" x2="3.81" y2="20.32" width="0.4064" layer="1"/>
@@
 <wire x1="27.94" y1="3.81" x2="33.782" y2="9.652" width="0.4064" layer="1"/>
 <wire x1="33.782" y1="9.652" x2="33.782" y2="33.274" width="0.4064" layer="1"/>
-<wire x1="33.782" y1="33.274" x2="28.956" y2="38.1" width="0.4064" layer="1"/>
-<via x="25.146" y="38.1" extent="1-16" drill="0.8"/>
-<wire x1="11.51395" y1="24.296" x2="25.31795" y2="38.1" width="0.4064" layer="1"/>
-<wire x1="25.146" y1="38.1" x2="25.31795" y2="38.1" width="0.4064" layer="1"/>
-<wire x1="28.956" y1="38.1" x2="25.146" y2="38.1" width="0.4064" layer="1"/>
+<wire x1="28.956" y1="38.1" x2="33.782" y2="33.274" width="0.4064" layer="1"/>
+<via x="20.828" y="38.1" extent="1-16" drill="1"/>
+<wire x1="11.51395" y1="24.296" x2="20.786975" y2="33.569025" width="0.4064" layer="1"/>
+<wire x1="20.828" y1="38.1" x2="20.828" y2="33.61005" width="0.4064" layer="1"/>
+<wire x1="20.828" y1="33.61005" x2="20.786975" y2="33.569025" width="0.4064" layer="1"/>
+<wire x1="20.828" y1="38.1" x2="28.956" y2="38.1" width="0.4064" layer="1"/>
 </signal>
 <signal name="N$3">
@@
 <wire x1="26.67" y1="30.988" x2="25.466" y2="32.192" width="0.4064" layer="1"/>
 <wire x1="25.466" y1="32.192" x2="25.466" y2="32.766" width="0.4064" layer="1"/>
+<contactref element="R6_2" pad="1"/>
+<wire x1="25.466" y1="36.068" x2="25.466" y2="32.766" width="0.4064" layer="1"/>
 </signal>
 <signal name="N$5">
@@
 <wire x1="32.766" y1="31.75" x2="32.766" y2="16.676" width="0.4064" layer="1"/>
 <wire x1="32.766" y1="16.676" x2="30.314" y2="14.224" width="0.4064" layer="1"/>
+<contactref element="R6_2" pad="2"/>
+<wire x1="27.366" y1="36.068" x2="27.366" y2="32.766" width="0.4064" layer="1"/>
+<wire x1="27.366" y1="32.766" x2="27.432" y2="32.7" width="0.4064" layer="1"/>
 </signal>
 </signals>
